Commit message: Update task_board

File: task_board/task_board_description/urdf/task_board.urdf (robot description, URDF)
Before this commit: robot task_board, 1 links, 0 joints
Links:
- removed link shell
- added link task_board_hole_1; collision mesh filename=package://task_board_description/meshes/collision/task_boar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; collision mesh filename=package://task_board_description/meshes/collision/task_boar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
- added link task_board_hole_2; collision mesh filename=package://task_board_description/meshes/collision/task_boar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; collision mesh filename=package://task_board_description/meshes/collision/task_boar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
- added link task_board_hole_3; collision mesh filename=package://task_board_description/meshes/collision/task_boar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; collision mesh filename=package://task_board_description/meshes/collision/task_boar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
- added link task_board_lid; collision mesh filename=package://task_board_description/meshes/collision/task_boar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; visual mesh filename=package://task_board_description/meshes/visual/task_board_l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
- added link task_board_lid_knob; collision mesh filename=package://task_board_description/meshes/collision/task_boar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; visual mesh filename=package://task_board_description/meshes/visual/task_board_l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
- added link task_board_main; collision mesh filename=package://task_board_description/meshes/collision/task_boar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; collision mesh filename=package://task_board_description/meshes/collision/task_boar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
- added link task_board_slider; collision mesh filename=package://task_board_description/meshes/collision/task_boar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; visual mesh filename=package://task_board_description/meshes/visual/task_board_s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
Joints:
- added joint task_board_hole_1_joint: type fixed, parent task_board_main, child task_board_hole_1, origin xyz=-0.0191 0.039 0.0734 rpy=0 0 0
- added joint task_board_hole_2_joint: type fixed, parent task_board_main, child task_board_hole_2, origin xyz=-0.044 0.039 0.0734 rpy=0 0 0
- added joint task_board_hole_3_joint: type fixed, parent task_board_main, child task_board_hole_3, origin xyz=0.037334 -0.102 0.0963 rpy=0 ${-pi/2} 0
- added joint task_board_lid_joint: type continuous, parent task_board_main, child task_board_lid, origin xyz=0.033026 -0.0472 0.079405 rpy=0 0 0, axis 0 1 0
- added joint task_board_lid_knob_joint: type fixed, parent task_board_lid, child task_board_lid_knob, origin xyz=-0.066776 0.0 0.010587 rpy=0 0 0
- added joint task_board_slider_joint: type prismatic, parent task_board_main, child task_board_slider, origin xyz=0.04301 0.061594 0.082959 rpy=0 0 0, axis 1 0 0, limit lower=-0.025 upper=0.01 effort=1000 velocity=1000

Commit message: Update task_board

File: task_board/task_board_description/urdf/task_board.urdf (robot description, URDF)
Before this commit: robot task_board, 7 links, 6 joints
Links:
- added link task_board_button_1; collision mesh filename=package://task_board_description/meshes/collision/task_boar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; visual mesh filename=package://task_board_description/meshes/visual/task_board_b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
- added link task_board_button_2; collision mesh filename=package://task_board_description/meshes/collision/task_boar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; visual mesh filename=package://task_board_description/meshes/visual/task_board_b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
- added link task_board_clock; collision mesh filename=package://task_board_description/meshes/collision/task_boar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; visual mesh filename=package://task_board_description/meshes/visual/task_board_c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
- link task_board_lid: geometry collision mesh filename=package://task_board_description/meshes/collision/task_boar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; collision mesh filename=package://task_board_description/meshes/collision/task_boar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
- link task_board_lid_knob: geometry collision cylinder length=0.0027 radius=0.007486; collision cylinder length=0.006 radius=0.004
- link task_board_main: geometry collision mesh filename=package://task_board_description/meshes/collision/task_boar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; collision mesh filename=package://task_board_description/meshes/collision/task_boar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
Joints:
- added joint task_board_button_1_joint: type prismatic, parent task_board_main, child task_board_button_1, origin xyz=-0.043957 0.09625 0.0835 rpy=0 0 0, axis 0 0 1, limit lower=-0.003 upper=0 effort=1000 velocity=1000
- added joint task_board_button_2_joint: type prismatic, parent task_board_main, child task_board_button_2, origin xyz=-0.02995 0.09625 0.0835 rpy=0 0 0, axis 0 0 1, limit lower=-0.003 upper=0 effort=1000 velocity=1000
- added joint task_board_clock_joint: type fixed, parent task_board_main, child task_board_clock, origin xyz=0.02361 0.09598 0.086058 rpy=0 0 0
- joint task_board_hole_3_joint: origin xyz=0.037334 -0.102 0.0963 rpy=0 ${-pi/2} 0 -> xyz=0.037334 -0.102 0.0963 rpy=0 -1.5707963267948966 0
- joint task_board_lid_joint: limit (none) -> lower=0.0 upper=2.072927552593665 effort=1000 velocity=1000; type continuous -> revolute
