Commit message: Restructure task_board

File: task_board/urdf/task_board.urdf (robot description, URDF)
Before this commit: robot task_board, 10 links, 9 joints
Links:
- link task_board_button_1: geometry collision mesh filename=package://task_board/meshes/collision/task_board_button.stl; visual mesh filename=package://task_board/meshes/visual/task_board_button.dae
- link task_board_button_2: geometry collision mesh filename=package://task_board/meshes/collision/task_board_button.stl; visual mesh filename=package://task_board/meshes/visual/task_board_button.dae
- link task_board_clock: geometry collision mesh filename=package://task_board/meshes/collision/task_board_clock.stl; visual mesh filename=package://task_board/meshes/visual/task_board_clock.dae
- link task_board_hole_1: geometry collision mesh filename=package://task_board/meshes/collision/task_board_hole_side.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; collision mesh filename=package://task_board/meshes/collision/task_board_hole_side.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
- link task_board_hole_2: geometry collision mesh filename=package://task_board/meshes/collision/task_board_hole_side.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; collision mesh filename=package://task_board/meshes/collision/task_board_hole_side.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
- link task_board_hole_3: geometry collision mesh filename=package://task_board/meshes/collision/task_board_hole_side.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; collision mesh filename=package://task_board/meshes/collision/task_board_hole_side.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
- link task_board_lid: geometry collision mesh filename=package://task_board/meshes/collision/task_board_lid.stl; collision mesh filename=package://task_board/meshes/collision/task_board_lid_hinge.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
- link task_board_lid_knob: geometry collision cylinder length=0.0027 radius=0.007486; collision cylinder length=0.006 radius=0.004
- link task_board_main: geometry collision mesh filename=package://task_board/meshes/collision/task_board_part_1.stl; collision mesh filename=package://task_board/meshes/collision/task_board_part_10.stl
- link task_board_slider: geometry collision mesh filename=package://task_board/meshes/collision/task_board_slider.stl; visual mesh filename=package://task_board/meshes/visual/task_board_slider.dae
