Commit message: Update task_board

File: task_board/mjcf/task_board/stl/task_board.urdf (robot description, URDF)
Before this commit: robot task_board, 10 links, 9 joints
Links:
- link task_board_button_1: geometry collision mesh filename=task_board_button.stl; visual mesh filename=package://task_board/meshes/visual/task_board_button.dae
- link task_board_button_2: geometry collision mesh filename=task_board_button.stl; visual mesh filename=package://task_board/meshes/visual/task_board_button.dae
- link task_board_clock: geometry collision mesh filename=task_board_clock.stl; visual mesh filename=package://task_board/meshes/visual/task_board_clock.dae
- link task_board_hole_1: geometry collision mesh filename=task_board_hole_side.stl; collision mesh filename=task_board_hole_side.stl
- link task_board_hole_2: geometry collision mesh filename=task_board_hole_side.stl; collision mesh filename=task_board_hole_side.stl
- link task_board_hole_3: geometry collision mesh filename=task_board_hole_side.stl; collision mesh filename=task_board_hole_side.stl
- link task_board_lid: geometry collision mesh filename=task_board_lid.stl; collision mesh filename=task_board_lid_hinge.stl
- link task_board_lid_knob: geometry collision cylinder length=0.0027 radius=0.007486; collision cylinder length=0.006 radius=0.004
- link task_board_main: geometry collision mesh filename=task_board_part_1.stl; collision mesh filename=task_board_part_10.stl
- link task_board_slider: geometry collision mesh filename=task_board_slider.stl; visual mesh filename=package://task_board/meshes/visual/task_board_slider.dae
Joints:
- removed joint task_board_button_1_joint
- removed joint task_board_button_2_joint
- removed joint task_board_clock_joint
- removed joint task_board_hole_1_joint
- removed joint task_board_hole_2_joint
- removed joint task_board_hole_3_joint
- removed joint task_board_lid_joint
- removed joint task_board_lid_knob_joint
- removed joint task_board_slider_joint
- added joint task_board_button_1_joint_0: type prismatic, parent task_board_main, child task_board_button_1, origin xyz=-0.043957 0.09625 0.0835 rpy=0 0 0, axis 0 0 1, limit lower=-0.003 upper=0 effort=1000 velocity=1000
- added joint task_board_button_2_joint_0: type prismatic, parent task_board_main, child task_board_button_2, origin xyz=-0.02995 0.09625 0.0835 rpy=0 0 0, axis 0 0 1, limit lower=-0.003 upper=0 effort=1000 velocity=1000
- added joint task_board_clock_joint_0: type fixed, parent task_board_main, child task_board_clock, origin xyz=0.02361 0.09598 0.086058 rpy=0 0 0
- added joint task_board_hole_1_joint_0: type fixed, parent task_board_main, child task_board_hole_1, origin xyz=-0.0191 0.039 0.0734 rpy=0 0 0
- added joint task_board_hole_2_joint_0: type fixed, parent task_board_main, child task_board_hole_2, origin xyz=-0.044 0.039 0.0734 rpy=0 0 0
- added joint task_board_hole_3_joint_0: type fixed, parent task_board_main, child task_board_hole_3, origin xyz=0.037334 -0.102 0.0963 rpy=0 -1.5707963267948966 0
- added joint task_board_lid_joint_0: type revolute, parent task_board_main, child task_board_lid, origin xyz=0.033026 -0.0472 0.079405 rpy=0 0 0, axis 0 1 0, limit lower=0.0 upper=2.072927552593665 effort=1000 velocity=1000
- added joint task_board_lid_knob_joint_0: type fixed, parent task_board_lid, child task_board_lid_knob, origin xyz=-0.066776 0.0 0.010587 rpy=0 0 0
- added joint task_board_slider_joint_0: type prismatic, parent task_board_main, child task_board_slider, origin xyz=0.04301 0.061594 0.082959 rpy=0 0 0, axis 1 0 0, limit lower=-0.025 upper=0.01 effort=1000 velocity=1000

File: task_board/urdf/task_board.urdf (robot description, URDF)
Before this commit: robot task_board, 10 links, 9 joints
Joints:
- removed joint task_board_button_1_joint
- removed joint task_board_button_2_joint
- removed joint task_board_clock_joint
- removed joint task_board_hole_1_joint
- removed joint task_board_hole_2_joint
- removed joint task_board_hole_3_joint
- removed joint task_board_lid_joint
- removed joint task_board_lid_knob_joint
- removed joint task_board_slider_joint
- added joint task_board_button_1_joint_0: type prismatic, parent task_board_main, child task_board_button_1, origin xyz=-0.043957 0.09625 0.0835 rpy=0 0 0, axis 0 0 1, limit lower=-0.003 upper=0 effort=1000 velocity=1000
- added joint task_board_button_2_joint_0: type prismatic, parent task_board_main, child task_board_button_2, origin xyz=-0.02995 0.09625 0.0835 rpy=0 0 0, axis 0 0 1, limit lower=-0.003 upper=0 effort=1000 velocity=1000
- added joint task_board_clock_joint_0: type fixed, parent task_board_main, child task_board_clock, origin xyz=0.02361 0.09598 0.086058 rpy=0 0 0
- added joint task_board_hole_1_joint_0: type fixed, parent task_board_main, child task_board_hole_1, origin xyz=-0.0191 0.039 0.0734 rpy=0 0 0
- added joint task_board_hole_2_joint_0: type fixed, parent task_board_main, child task_board_hole_2, origin xyz=-0.044 0.039 0.0734 rpy=0 0 0
- added joint task_board_hole_3_joint_0: type fixed, parent task_board_main, child task_board_hole_3, origin xyz=0.037334 -0.102 0.0963 rpy=0 -1.5707963267948966 0
- added joint task_board_lid_joint_0: type revolute, parent task_board_main, child task_board_lid, origin xyz=0.033026 -0.0472 0.079405 rpy=0 0 0, axis 0 1 0, limit lower=0.0 upper=2.072927552593665 effort=1000 velocity=1000
- added joint task_board_lid_knob_joint_0: type fixed, parent task_board_lid, child task_board_lid_knob, origin xyz=-0.066776 0.0 0.010587 rpy=0 0 0
- added joint task_board_slider_joint_0: type prismatic, parent task_board_main, child task_board_slider, origin xyz=0.04301 0.061594 0.082959 rpy=0 0 0, axis 1 0 0, limit lower=-0.025 upper=0.01 effort=1000 velocity=1000

Commit message: Fix task_board

File: task_board/mjcf/task_board/stl/task_board.urdf (robot description, URDF)
Before this commit: robot task_board, 10 links, 9 joints
Joints:
- removed joint task_board_button_1_joint_0
- removed joint task_board_button_2_joint_0
- removed joint task_board_clock_joint_0
- removed joint task_board_hole_1_joint_0
- removed joint task_board_hole_2_joint_0
- removed joint task_board_hole_3_joint_0
- removed joint task_board_lid_joint_0
- removed joint task_board_lid_knob_joint_0
- removed joint task_board_slider_joint_0
- added joint task_board_button_1_joint: type prismatic, parent task_board_main, child task_board_button_1, origin xyz=-0.043957 0.09625 0.0835 rpy=0 0 0, axis 0 0 1, limit lower=-0.003 upper=0 effort=1000 velocity=1000
- added joint task_board_button_2_joint: type prismatic, parent task_board_main, child task_board_button_2, origin xyz=-0.02995 0.09625 0.0835 rpy=0 0 0, axis 0 0 1, limit lower=-0.003 upper=0 effort=1000 velocity=1000
- added joint task_board_clock_joint: type fixed, parent task_board_main, child task_board_clock, origin xyz=0.02361 0.09598 0.086058 rpy=0 0 0
- added joint task_board_hole_1_joint: type fixed, parent task_board_main, child task_board_hole_1, origin xyz=-0.0191 0.039 0.0734 rpy=0 0 0
- added joint task_board_hole_2_joint: type fixed, parent task_board_main, child task_board_hole_2, origin xyz=-0.044 0.039 0.0734 rpy=0 0 0
- added joint task_board_hole_3_joint: type fixed, parent task_board_main, child task_board_hole_3, origin xyz=0.037334 -0.102 0.0963 rpy=0 -1.5707963267948966 0
- added joint task_board_lid_joint: type revolute, parent task_board_main, child task_board_lid, origin xyz=0.033026 -0.0472 0.079405 rpy=0 0 0, axis 0 1 0, limit lower=0.0 upper=2.072927552593665 effort=1000 velocity=1000
- added joint task_board_lid_knob_joint: type fixed, parent task_board_lid, child task_board_lid_knob, origin xyz=-0.066776 0.0 0.010587 rpy=0 0 0
- added joint task_board_slider_joint: type prismatic, parent task_board_main, child task_board_slider, origin xyz=0.04301 0.061594 0.082959 rpy=0 0 0, axis 1 0 0, limit lower=-0.025 upper=0.01 effort=1000 velocity=1000

File: task_board/urdf/task_board.urdf (robot description, URDF)
Before this commit: robot task_board, 10 links, 9 joints
Joints:
- removed joint task_board_button_1_joint_0
- removed joint task_board_button_2_joint_0
- removed joint task_board_clock_joint_0
- removed joint task_board_hole_1_joint_0
- removed joint task_board_hole_2_joint_0
- removed joint task_board_hole_3_joint_0
- removed joint task_board_lid_joint_0
- removed joint task_board_lid_knob_joint_0
- removed joint task_board_slider_joint_0
- added joint task_board_button_1_joint: type prismatic, parent task_board_main, child task_board_button_1, origin xyz=-0.043957 0.09625 0.0835 rpy=0 0 0, axis 0 0 1, limit lower=-0.003 upper=0 effort=1000 velocity=1000
- added joint task_board_button_2_joint: type prismatic, parent task_board_main, child task_board_button_2, origin xyz=-0.02995 0.09625 0.0835 rpy=0 0 0, axis 0 0 1, limit lower=-0.003 upper=0 effort=1000 velocity=1000
- added joint task_board_clock_joint: type fixed, parent task_board_main, child task_board_clock, origin xyz=0.02361 0.09598 0.086058 rpy=0 0 0
- added joint task_board_hole_1_joint: type fixed, parent task_board_main, child task_board_hole_1, origin xyz=-0.0191 0.039 0.0734 rpy=0 0 0
- added joint task_board_hole_2_joint: type fixed, parent task_board_main, child task_board_hole_2, origin xyz=-0.044 0.039 0.0734 rpy=0 0 0
- added joint task_board_hole_3_joint: type fixed, parent task_board_main, child task_board_hole_3, origin xyz=0.037334 -0.102 0.0963 rpy=0 -1.5707963267948966 0
- added joint task_board_lid_joint: type revolute, parent task_board_main, child task_board_lid, origin xyz=0.033026 -0.0472 0.079405 rpy=0 0 0, axis 0 1 0, limit lower=0.0 upper=2.072927552593665 effort=1000 velocity=1000
- added joint task_board_lid_knob_joint: type fixed, parent task_board_lid, child task_board_lid_knob, origin xyz=-0.066776 0.0 0.010587 rpy=0 0 0
- added joint task_board_slider_joint: type prismatic, parent task_board_main, child task_board_slider, origin xyz=0.04301 0.061594 0.082959 rpy=0 0 0, axis 1 0 0, limit lower=-0.025 upper=0.01 effort=1000 velocity=1000
