Commit message: Add static_objects

File: articulated_objects/box/urdf/box.urdf (robot description, URDF)
Before this commit: robot box, 3 links, 2 joints
Links:
- link box: mass 2.789491653442383 -> None; geometry visual box size=0.005156 0.32 0.335; visual box size=0.005156 0.32 0.335
- link box_flap_side_1: mass 0.2165265679359436 -> None; geometry visual mesh filename=package://articulated_objects/box/meshes/stl/BoxFlapSide1.s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
- link box_flap_side_2: mass 0.2165265679359436 -> None; geometry visual mesh filename=package://articulated_objects/box/meshes/stl/BoxFlapSide2.s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
Joints:
- joint box_flap_side_1_joint: limit lower=-3.14 upper=3.14 effort=1000 velocity=1000 -> lower=-1.57 upper=4.7 effort=1000.0 velocity=3.1415; origin xyz=0.17000000178813934 0.0 0.16599999368190765 rpy=0.0 -0.0 0.0 -> xyz=0.17 0 0.166 rpy=0 0 0
- joint box_flap_side_2_joint: limit lower=-3.14 upper=3.14 effort=1000 velocity=1000 -> lower=-1.57 upper=4.7 effort=1000.0 velocity=3.1415; origin xyz=-0.17000000178813934 0.0 0.1679999977350235 rpy=0.0 -0.0 0.0 -> xyz=-0.17 0 0.168 rpy=0 0 0

Commit message: Update box

File: articulated_objects/box/urdf/box.urdf (robot description, URDF)
Before this commit: robot box, 3 links, 2 joints
Links:
- link box: geometry collision box size=0.005156 0.32 0.335; collision box size=0.005156 0.32 0.335
- link box_flap_side_1: geometry collision mesh filename=package://articulated_objects/box/meshes/stl/BoxFlapSide1.s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; visual mesh filename=package://articulated_objects/box/meshes/stl/BoxFlapSide1.s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
- link box_flap_side_2: geometry collision mesh filename=package://articulated_objects/box/meshes/stl/BoxFlapSide2.s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; visual mesh filename=package://articulated_objects/box/meshes/stl/BoxFlapSide2.s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
